Commit message: added fkin

File: basic134/urdf/threedofexample.urdf (robot description, URDF)
Before this commit: robot threedofexample, 9 links, 8 joints
Joints:
- joint lbracket: origin xyz=0 0.05 0.123 rpy=0 -1.5708 1.5708 -> xyz=0 0.05 0.13 rpy=0 -1.5708 1.5708

Commit message: Midterm push

File: basic134/urdf/threedofexample.urdf (robot description, URDF)
Before this commit: robot threedofexample, 9 links, 8 joints
Joints:
- joint baseplate: origin xyz=0 0 0.0230 rpy=0 0 -1.5708 -> xyz=-0.0145 .016 0.0095 rpy=0 0 -1.5708
- joint lbracket: origin xyz=0 0.05 0.13 rpy=0 -1.5708 1.5708 -> xyz=0.0 0.05 0.13 rpy=0 -1.5708 1.5708
