Commit message: bmo finished

File: bmoHanoi/urdf/sixDOFold.urdf (robot description, URDF)
Before this commit: robot sixDOF, 12 links, 11 joints
Links:
- removed link claw
- removed link lbracket
- added link bruh
- link baseplate: geometry visual box size=0.2 0.1 0.0450
Joints:
- removed joint claw
- removed joint lbracket
- added joint temptoCam: type fixed, parent bruh, child camera, origin xyz=-.033 .078 -.017 rpy=0 0 0
- joint base: child lbracket -> shouldermotor; origin xyz=0 0 0.054 rpy=0 0 0 -> xyz=0.032 0 0.0625 rpy=0 0 1.5708
- joint baseplate: origin xyz=0 0.0745 0.0230 rpy=0 0 0 -> xyz=0 0 0.0450 rpy=0 0 1.5708
- joint elbow: origin xyz=-0.0575 0 0 rpy=0 0 3.1415 -> xyz=-0.056 0 0 rpy=0 0 3.1415
- joint elbowBase: origin xyz=0 0 .448 rpy=0 0 0 -> xyz=0 0 .452 rpy=0 0 0
- joint final: origin xyz=.0085 .075 -.0075 rpy=0 0 0 -> xyz=.033 .0655  -.0117 rpy=0 0 0
- joint head: child claw -> bruh; origin xyz=-.09 0 -.045 rpy=0 0 0 -> xyz=-.044 0 -.092 rpy=0 0 0
- joint shoulder: origin xyz=0 0 0.0 rpy=0 -1.5708 0 -> xyz=0 0 0.0 rpy=3.14159 3.14159 0
- joint wrist: origin xyz=0 0 .448 rpy=0 0 0 -> xyz=-.048 0 .451 rpy=0 0 0
