Commit message: states

File: bmoHanoi/urdf/sixDOF.urdf (robot description, URDF)
Before this commit: robot sixDOF, 7 links, 6 joints
Links:
- added link donut
Joints:
- added joint claw: type continuous, parent hand, child camera, origin xyz=-.0975 0 -.045 rpy=0 0 0, axis 0 0 -1
- added joint gripper: type fixed, parent tip, child donut, origin xyz=.035 .095 -0.08 rpy=0 0 0

Commit message: implemented grabbing

File: bmoHanoi/urdf/sixDOF.urdf (robot description, URDF)
Before this commit: robot sixDOF, 8 links, 8 joints
Links:
- removed link donut
- added link basemotor; visual mesh filename=package://bmoHanoi/meshes/X8.stl scale=0.001 0.001 0.001
- added link baseplate; visual box size=0.2 0.1 0.0230
- added link claw; visual mesh filename=package://bmoHanoi/meshes/BMOClaw.stl scale=0.001 0.001 0.001
- added link elbowmotor; visual mesh filename=package://bmoHanoi/meshes/X8.stl scale=0.001 0.001 0.001
- added link shouldermotor; visual mesh filename=package://bmoHanoi/meshes/X8.stl scale=0.001 0.001 0.001
- link bicep: geometry visual mesh filename=package://bmoHanoi/meshes/BMOArm.stl scale=0.001 0.001 0.001
- link forearm: geometry visual mesh filename=package://bmoHanoi/meshes/BMOArm.stl scale=0.001 0.001 0.001
Joints:
- removed joint gripper
- added joint baseplate: type fixed, parent baseplate, child basemotor, origin xyz=0 0 0.0230 rpy=0 0 0
- added joint elbowBase: type fixed, parent bicep, child elbowmotor, origin xyz=0 0 .4351 rpy=0 0 0, axis 1 0 0 
- added joint lbracket: type fixed, parent lbracket, child shouldermotor, origin xyz=-0.02 0 0.045 rpy=0 1.5708 0
- added joint placement: type fixed, parent world, child baseplate, origin xyz=0 0 0 rpy=0 0 0
- joint base: origin xyz=0 -.0775 0.07 rpy=0 0 0 -> xyz=0 0 0.0451 rpy=0 0 0; parent world -> basemotor
- joint claw: axis 0 0 -1 -> (none); origin xyz=-.0975 0 -.045 rpy=0 0 0 -> xyz=-.03 .095 -0.02 rpy=0 0 0; parent hand -> claw; type continuous -> fixed
- joint elbow: origin xyz=0.052 0 .45 rpy=0 0 0 -> xyz=-0.0512 0 0 rpy=0 0 3.1415; parent bicep -> elbowmotor
- joint final: origin xyz=.035 .095 -0.08 rpy=0 0 0 -> xyz=.035 .035 -0.09 rpy=0 0 0
- joint head: child camera -> claw
- joint shoulder: axis -1 0 0 -> 1 0 0; origin xyz=0 0 .055 rpy=0 0 0 -> xyz=0 0 0.0512 rpy=0 -1.5708 0; parent lbracket -> shouldermotor

Commit message: BMO picks up from pegs

File: bmoHanoi/urdf/sixDOF.urdf (robot description, URDF)
Before this commit: robot sixDOF, 12 links, 11 joints
Joints:
- joint final: origin xyz=.035 .035 -0.09 rpy=0 0 0 -> xyz=.035 .07 -0.065 rpy=0 0 0

Commit message: added priorities, need to figure out game states

File: bmoHanoi/urdf/sixDOF.urdf (robot description, URDF)
Before this commit: robot sixDOF, 12 links, 11 joints
Joints:
- joint final: origin xyz=.035 .07 -0.065 rpy=0 0 0 -> xyz=.035 .07 -0.035 rpy=0 0 0

Commit message: got bmo with the new urdf and valid grabs 10/10 times

File: bmoHanoi/urdf/sixDOF.urdf (robot description, URDF)
Before this commit: robot sixDOF, 12 links, 11 joints
Links:
- removed link claw
- removed link lbracket
- added link bruh
- link baseplate: geometry visual box size=0.2 0.1 0.0450
Joints:
- removed joint claw
- removed joint lbracket
- added joint temptoCam: type fixed, parent bruh, child camera, origin xyz=-.033 .078 -.017 rpy=0 0 0
- joint base: child lbracket -> shouldermotor; origin xyz=0 0 0.0451 rpy=0 0 0 -> xyz=0.032 0 0.0625 rpy=0 0 1.5708
- joint baseplate: origin xyz=0 0 0.0230 rpy=0 0 0 -> xyz=0 0 0.0450 rpy=0 0 1.5708
- joint elbow: origin xyz=-0.0512 0 0 rpy=0 0 3.1415 -> xyz=-0.056 0 0 rpy=0 0 3.1415
- joint elbowBase: origin xyz=0 0 .4351 rpy=0 0 0 -> xyz=0 0 .452 rpy=0 0 0
- joint final: origin xyz=.035 .07 -0.065 rpy=0 0 0 -> xyz=.033 .063  -.01 rpy=0 0 0
- joint head: child claw -> bruh; origin xyz=-.0975 0 -.045 rpy=0 0 0 -> xyz=-.044 0 -.092 rpy=0 0 0
- joint shoulder: origin xyz=0 0 0.0512 rpy=0 -1.5708 0 -> xyz=0 0 0.0 rpy=3.14159 3.14159 0
- joint wrist: origin xyz=0 0 .465 rpy=0 0 0 -> xyz=-.048 0 .451 rpy=0 0 0

Commit message: trying a new honing method??

File: bmoHanoi/urdf/sixDOF.urdf (robot description, URDF)
Before this commit: robot sixDOF, 11 links, 10 joints
Joints:
- joint final: origin xyz=.033 .063  -.01 rpy=0 0 0 -> xyz=.033 .058  -.0195 rpy=0 0 0

Commit message: starting game states pt2

File: bmoHanoi/urdf/sixDOF.urdf (robot description, URDF)
Before this commit: robot sixDOF, 11 links, 10 joints
Joints:
- joint final: origin xyz=.033 .058  -.0195 rpy=0 0 0 -> xyz=.033 .048  -.0095 rpy=0 0 0

Commit message: worked w jordo about to start bit decoding

File: bmoHanoi/urdf/sixDOF.urdf (robot description, URDF)
Before this commit: robot sixDOF, 12 links, 11 joints
Joints:
- joint final: origin xyz=.0085 .075 -.0075 rpy=0 0 0 -> xyz=.0005 .08 -.0210 rpy=0 0 0

Commit message: everything is broken

File: bmoHanoi/urdf/sixDOF.urdf (robot description, URDF)
Before this commit: robot sixDOF, 12 links, 11 joints
Joints:
- joint final: origin xyz=.0005 .08 -.0210 rpy=0 0 0 -> xyz=.0005 .08 -.0110 rpy=0 0 0

Commit message: ITS OVERRRRR

File: bmoHanoi/urdf/sixDOF.urdf (robot description, URDF)
Before this commit: robot sixDOF, 12 links, 11 joints
Joints:
- joint final: origin xyz=.0005 .08 -.0110 rpy=0 0 0 -> xyz=.0125 .08 -.0110 rpy=0 0 0
